Commit message: add grasp point

File: robotiq_description/urdf/robotiq_gripper_macro.urdf.xacro (robot description, xacro)
@@ -139,4 +139,5 @@
             </inertial>
         </link>
+        <link name="${prefix}robotiq_grasp_point"/>
         <link name="${prefix}robotiq_85_right_finger_tip_link">
             <visual>
@@ -213,4 +214,9 @@
             <origin xyz="-0.00563134 0.0 0.04718515" rpy="0 0 0" />
             <mimic joint="${prefix}robotiq_85_left_knuckle_joint" />
+        </joint>
+        <joint name="${prefix}robotiq_grasp_point_tip_joint" type="fixed">
+            <parent link="${prefix}robotiq_85_base_link" />
+            <child link="${prefix}robotiq_grasp_point" />
+            <origin xyz="0.0 0.0 0.15" rpy="0 0 0" />
         </joint>
         <xacro:if value="${sim}">

Commit message: add mujoco

File: robotiq_description/urdf/robotiq_gripper_macro.urdf.xacro (robot description, xacro)
@@ -2,5 +2,5 @@
 <robot xmlns:xacro="http://wiki.ros.org/xacro" name="robotiq_gripper">
     <xacro:include filename="$(find robotiq_description)/urdf/robotiq_sim_gripper.ros2_control.xacro"/>
-    <xacro:macro name="robotiq_gripper" params="parent *origin sim:=false prefix">
+    <xacro:macro name="robotiq_gripper" params="parent *origin sim:=false prefix mujoco_model sim_mujoco">
         <link name="${prefix}robotiq_85_base_link">
             <visual>
@@ -221,5 +221,5 @@
         </joint>
         <xacro:if value="${sim}">
-            <xacro:robotiq_sim_gripper_ros2_control name="ros2_sim_control" sim_isaac="false" sim_ignition="true" use_fake_hardware="false">
+            <xacro:robotiq_sim_gripper_ros2_control name="ros2_sim_control" sim_isaac="false" sim_ignition="false" use_fake_hardware="false" sim_mujoco="true" mujoco_model="${mujoco_model}">
             </xacro:robotiq_sim_gripper_ros2_control>
             <gazebo reference="${prefix}robotiq_85_right_finger_tip_link">

File: robotiq_description/urdf/robotiq_sim_gripper.ros2_control.xacro (robot description, xacro)
@@ -2,5 +2,5 @@
 <robot xmlns:xacro="http://www.ros.org/wiki/xacro">
     <xacro:macro name="robotiq_sim_gripper_ros2_control"
-                 params="name sim_ignition:=false sim_isaac:=false use_fake_hardware:=true">
+                 params="name sim_ignition:=false sim_isaac:=false use_fake_hardware:=true sim_mujoco:=false, mujoco_model">
         <ros2_control name="${name}" type="system">
             <!-- Plugins -->
@@ -18,4 +18,8 @@
                     <param name="fake_sensor_commands">${fake_sensor_commands}</param>
                     <param name="state_following_offset">0.0</param>
+                </xacro:if>
+                <xacro:if value="${sim_mujoco}">
+                    <plugin>cartesian_controller_simulation/Simulator</plugin>
+                    <param name="mujoco_model">${mujoco_model}</param>
                 </xacro:if>
             </hardware>
@@ -81,5 +85,5 @@
             </joint>
             <!-- Only add this with fake hardware mode -->
-            <xacro:unless value="${sim_ignition or sim_isaac}">
+            <xacro:unless value="${sim_ignition or sim_isaac or sim_mujoco}">
                 <gpio name="reactivate_gripper">
                     <command_interface name="reactivate_gripper_cmd" />

Commit message: fix args in xacro

File: robotiq_description/urdf/robotiq_gripper_macro.urdf.xacro (robot description, xacro)
@@ -2,5 +2,5 @@
 <robot xmlns:xacro="http://wiki.ros.org/xacro" name="robotiq_gripper">
     <xacro:include filename="$(find robotiq_description)/urdf/robotiq_sim_gripper.ros2_control.xacro"/>
-    <xacro:macro name="robotiq_gripper" params="parent *origin sim:=false prefix mujoco_model sim_mujoco">
+    <xacro:macro name="robotiq_gripper" params="parent *origin sim:=false prefix mujoco_model sim_mujoco sim_gazebo use_fake_hardware:=true">
         <link name="${prefix}robotiq_85_base_link">
             <visual>
@@ -221,5 +221,5 @@
         </joint>
         <xacro:if value="${sim}">
-            <xacro:robotiq_sim_gripper_ros2_control name="ros2_sim_control" sim_isaac="false" sim_ignition="false" use_fake_hardware="false" sim_mujoco="true" mujoco_model="${mujoco_model}">
+            <xacro:robotiq_sim_gripper_ros2_control name="ros2_sim_control" sim_isaac="false" sim_gazebo="${sim_gazebo}" use_fake_hardware="${use_fake_hardware}" sim_mujoco="${sim_mujoco}" mujoco_model="${mujoco_model}">
             </xacro:robotiq_sim_gripper_ros2_control>
             <gazebo reference="${prefix}robotiq_85_right_finger_tip_link">

File: robotiq_description/urdf/robotiq_sim_gripper.ros2_control.xacro (robot description, xacro)
@@ -2,5 +2,5 @@
 <robot xmlns:xacro="http://www.ros.org/wiki/xacro">
     <xacro:macro name="robotiq_sim_gripper_ros2_control"
-                 params="name sim_ignition:=false sim_isaac:=false use_fake_hardware:=true sim_mujoco:=false, mujoco_model">
+                 params="name sim_gazebo:=false sim_isaac:=false use_fake_hardware:=true sim_mujoco:=false, mujoco_model">
         <ros2_control name="${name}" type="system">
             <!-- Plugins -->
@@ -11,11 +11,9 @@
                     <param name="joint_states_topic">/isaac_joint_states</param>
                 </xacro:if>
-                <xacro:if value="${sim_ignition}">
+                <xacro:if value="${sim_gazebo}">
                     <plugin>ign_ros2_control/IgnitionSystem</plugin>
                 </xacro:if>
                 <xacro:if value="${use_fake_hardware}">
                     <plugin>mock_components/GenericSystem</plugin>
-                    <param name="fake_sensor_commands">${fake_sensor_commands}</param>
-                    <param name="state_following_offset">0.0</param>
                 </xacro:if>
                 <xacro:if value="${sim_mujoco}">
@@ -27,10 +25,10 @@
             <joint name="robotiq_85_left_knuckle_joint">
                 <!-- With Ignition, we have mimic joints, so we only need this command interface activated -->
-                <xacro:if value="${sim_ignition}">
+                <xacro:if value="${sim_gazebo}">
                     <state_interface name="position">
                         <param name="initial_value">0.2</param>
                     </state_interface>
                 </xacro:if>
-                <xacro:unless value="${sim_ignition}">
+                <xacro:unless value="${sim_gazebo}">
                     <param name="initial_position">0.7929</param>
                     <state_interface name="position"/>
@@ -42,5 +40,5 @@
                 <param name="mimic">robotiq_85_left_knuckle_joint</param>
                 <param name="multiplier">-1</param>
-                <xacro:unless value="${sim_ignition}">
+                <xacro:unless value="${sim_gazebo}">
                     <command_interface name="position"/>
                     <state_interface name="position"/>
@@ -51,5 +49,5 @@
                 <param name="mimic">robotiq_85_left_knuckle_joint</param>
                 <param name="multiplier">1</param>
-                <xacro:unless value="${sim_ignition}">
+                <xacro:unless value="${sim_gazebo}">
                     <command_interface name="position"/>
                     <state_interface name="position"/>
@@ -60,5 +58,5 @@
                 <param name="mimic">robotiq_85_left_knuckle_joint</param>
                 <param name="multiplier">-1</param>
-                <xacro:unless value="${sim_ignition}">
+                <xacro:unless value="${sim_gazebo}">
                     <command_interface name="position"/>
                     <state_interface name="position"/>
@@ -69,5 +67,5 @@
                 <param name="mimic">robotiq_85_left_knuckle_joint</param>
                 <param name="multiplier">-1</param>
-                <xacro:unless value="${sim_ignition}">
+                <xacro:unless value="${sim_gazebo}">
                     <command_interface name="position"/>
                     <state_interface name="position"/>
@@ -78,5 +76,5 @@
                 <param name="mimic">robotiq_85_left_knuckle_joint</param>
                 <param name="multiplier">1</param>
-                <xacro:unless value="${sim_ignition}">
+                <xacro:unless value="${sim_gazebo}">
                     <command_interface name="position"/>
                     <state_interface name="position"/>
@@ -85,5 +83,5 @@
             </joint>
             <!-- Only add this with fake hardware mode -->
-            <xacro:unless value="${sim_ignition or sim_isaac or sim_mujoco}">
+            <xacro:unless value="${sim_gazebo or sim_isaac or sim_mujoco}">
                 <gpio name="reactivate_gripper">
                     <command_interface name="reactivate_gripper_cmd" />
